File: td4/logic.kicad_sch (KiCad schematic)
At the start: 33 parts, among them SW1 SW_DIP_x04, U1 74HC74, U10 74LS10, U2 74LS161, U3 74LS161, U4 74LS161, U5 74LS161, U6 74HC153, U7 74HC153, U8 74LS32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

Commit message: fix U5
Connections:
- net +3.3V: now also U5.10 (ENT), U5.7 (ENP)
- net GND: no longer U5.10 (ENT), U5.7 (ENP)
Changed lines of the file:
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@@
   (junction (at 203.2 167.64) (diameter 0) (color 0 0 0 0)
   )
-  (junction (at 100.33 262.89) (diameter 0) (color 0 0 0 0)
+  (junction (at 92.71 234.95) (diameter 0) (color 0 0 0 0)
   )
   (junction (at 58.42 143.51) (diameter 0) (color 0 0 0 0)
@@
   )
   (junction (at 110.49 222.25) (diameter 0) (color 0 0 0 0)
-  )
-  (junction (at 92.71 237.49) (diameter 0) (color 0 0 0 0)
   )
   (junction (at 193.04 121.92) (diameter 0) (color 0 0 0 0)
@@
     (stroke (width 0) (type default))
   )
-  (wire (pts (xy 92.71 234.95) (xy 92.71 237.49))
-    (stroke (width 0) (type default))
-  )
   (wire (pts (xy 293.37 48.26) (xy 279.4 48.26))
     (stroke (width 0) (type default))
@@
     (stroke (width 0) (type default))
   )
-  (wire (pts (xy 92.71 237.49) (xy 92.71 262.89))
-    (stroke (width 0) (type default))
-  )
   (wire (pts (xy 88.9 16.51) (xy 314.96 16.51))
     (stroke (width 0) (type default))
@@
     (stroke (width 0) (type default))
   )
-  (wire (pts (xy 92.71 262.89) (xy 100.33 262.89))
-    (stroke (width 0) (type default))
-  )
   (wire (pts (xy 58.42 251.46) (xy 97.79 251.46))
     (stroke (width 0) (type default))
@@
     (stroke (width 0) (type default))
   )
-  (wire (pts (xy 100.33 262.89) (xy 110.49 262.89))
-    (stroke (width 0) (type default))
-  )
   (wire (pts (xy 100.33 154.94) (xy 110.49 154.94))
     (stroke (width 0) (type default))
@@
     (stroke (width 0) (type default))
   )
+  (wire (pts (xy 92.71 222.25) (xy 110.49 222.25))
+    (stroke (width 0) (type default))
+  )
   (wire (pts (xy 161.29 274.32) (xy 161.29 276.86))
     (stroke (width 0) (type default))
   )
+  (wire (pts (xy 92.71 237.49) (xy 92.71 234.95))
+    (stroke (width 0) (type default))
+  )
   (wire (pts (xy 156.21 274.32) (xy 161.29 274.32))
     (stroke (width 0) (type default))
@@
   )
   (wire (pts (xy 252.73 186.69) (xy 339.09 186.69))
+    (stroke (width 0) (type default))
+  )
+  (wire (pts (xy 92.71 234.95) (xy 92.71 222.25))
     (stroke (width 0) (type default))
   )
@@
     )
   )
-  (symbol (lib_id "power:GND") (at 100.33 262.89 0) (unit 1)
+  (symbol (lib_id "power:GND") (at 110.49 262.89 0) (unit 1)
     (in_bom yes) (on_board yes) (dnp no) (fields_autoplaced)
-    (property "Reference" "#PWR09" (at 100.33 269.24 0)
+    (property "Reference" "#PWR09" (at 110.49 269.24 0)
       (effects (font (size 1.27 1.27)) hide)
     )
-    (property "Value" "GND" (at 100.33 267.97 0)
+    (property "Value" "GND" (at 110.49 267.97 0)
       (effects (font (size 1.27 1.27)))
     )
-    (property "Footprint" "" (at 100.33 262.89 0)
+    (property "Footprint" "" (at 110.49 262.89 0)
       (effects (font (size 1.27 1.27)) hide)
     )
-    (property "Datasheet" "" (at 100.33 262.89 0)
+    (property "Datasheet" "" (at 110.49 262.89 0)
       (effects (font (size 1.27 1.27)) hide)
     )
