File: td4/td4.kicad_pcb (KiCad board)
At the start: 2 copper layers, 137.2 x 76.2 mm, 55 parts, among them SW1 SW_DIP_x04, U0 Pico, U1 74HC74, U10 74LS10, U13 74HC14, U2 74LS161, U3 74LS161, U4 74LS161, U5 74LS161, U6 74HC153, U7 74HC153, U8 74LS32, U9 74HC283

Commit message: fix U5
Parts:
- renumbered LED2 to locked, LED3 to locked, Normal/Manual to locked, RST to locked, LED1 to locked, LED4 to locked, 10Hz/1Hz to locked, M_CLK to locked
Connections:
- U5 pad 10: GND -> +3.3V
- U5 pad 7: GND -> +3.3V
Routing:
- net +3.3V: track 413.3 -> 484.3 mm, vias 0 -> 2
- net Net-(U4-QD): track 52.0 -> 117.6 mm, vias 0 -> 1
- net /clock_reset/RESET: track 80.1 -> 135.4 mm
- net Net-(U5-~{LOAD}): track 28.7 -> 76.0 mm
- net /logic/D7: track 89.1 -> 134.6 mm, vias 1 -> 0
- net Net-(U7-IC2): track 116.1 -> 158.9 mm
- net Net-(U4-~{LOAD}): track 37.5 -> 79.1 mm, vias 1 -> 2
- net /logic/D0: track 78.4 -> 45.3 mm
- net Net-(U2-D): track 93.6 -> 125.2 mm, vias 1 -> 2
- net Net-(U7-1Y): track 90.4 -> 60.2 mm
- net Net-(U10-Pad11): track 42.4 -> 68.7 mm
- net /clock_reset/CLOCK: track 90.9 -> 114.8 mm
- net Net-(U7-2Y): track 62.0 -> 40.7 mm, vias 0 -> 4
- net Net-(SW20-C): track 49.6 -> 70.4 mm, vias 1 -> 0
- net Net-(U2-C): track 91.4 -> 70.8 mm, vias 0 -> 3
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